File: sch/display/display.sch (KiCad schematic (older format))
At the start: 17 parts, among them IC1 MAX7219, P1 INPUT, P2 CONN_1, P3 CONN_1, P4 CONN_1, P5 CONN_1, P6 OUTPUT

Commit message: Happy with the display module now.  Not done gerbers/drill yet but layout is done incl. silk screen.
Parts:
- renumbered AFF1 to D1, AFF5 to D2, AFF2 to D3, AFF6 to D4, AFF3 to D5, AFF7 to D6, AFF4 to D7, AFF8 to D8
Changed lines of the file:
@@
 $EndComp
 $Comp
-L 7SEGMENTS AFF1
+L 7SEGMENTS D1
 U 1 1 53712D36
 P 1900 3400
-F 0 "AFF1" H 1900 3950 60  0000 C CNN
+F 0 "D1" H 1900 3950 60  0000 C CNN
 F 1 "7SEGMENTS" H 1900 2950 60  0000 C CNN
 F 2 "" H 1900 3400 60  0000 C CNN
@@
 SEGDP
 $Comp
-L 7SEGMENTS AFF5
+L 7SEGMENTS D2
 U 1 1 53712FA9
 P 4050 3400
-F 0 "AFF5" H 4050 3950 60  0000 C CNN
+F 0 "D2" H 4050 3950 60  0000 C CNN
 F 1 "7SEGMENTS" H 4050 2950 60  0000 C CNN
 F 2 "" H 4050 3400 60  0000 C CNN
@@
 SEGDP
 $Comp
-L 7SEGMENTS AFF2
+L 7SEGMENTS D3
 U 1 1 5371306A
 P 1900 4550
-F 0 "AFF2" H 1900 5100 60  0000 C CNN
+F 0 "D3" H 1900 5100 60  0000 C CNN
 F 1 "7SEGMENTS" H 1900 4100 60  0000 C CNN
 F 2 "" H 1900 4550 60  0000 C CNN
@@
 SEGDP
 $Comp
-L 7SEGMENTS AFF6
+L 7SEGMENTS D4
 U 1 1 53713082
 P 4050 4550
-F 0 "AFF6" H 4050 5100 60  0000 C CNN
+F 0 "D4" H 4050 5100 60  0000 C CNN
 F 1 "7SEGMENTS" H 4050 4100 60  0000 C CNN
 F 2 "" H 4050 4550 60  0000 C CNN
@@
 SEGDP
 $Comp
-L 7SEGMENTS AFF3
+L 7SEGMENTS D5
 U 1 1 5371316C
 P 1900 5700
-F 0 "AFF3" H 1900 6250 60  0000 C CNN
+F 0 "D5" H 1900 6250 60  0000 C CNN
 F 1 "7SEGMENTS" H 1900 5250 60  0000 C CNN
 F 2 "" H 1900 5700 60  0000 C CNN
@@
 SEGDP
 $Comp
-L 7SEGMENTS AFF7
+L 7SEGMENTS D6
 U 1 1 53713184
 P 4050 5700
-F 0 "AFF7" H 4050 6250 60  0000 C CNN
+F 0 "D6" H 4050 6250 60  0000 C CNN
 F 1 "7SEGMENTS" H 4050 5250 60  0000 C CNN
 F 2 "" H 4050 5700 60  0000 C CNN
@@
 SEGDP
 $Comp
-L 7SEGMENTS AFF4
+L 7SEGMENTS D7
 U 1 1 5371319C
 P 1900 6850
-F 0 "AFF4" H 1900 7400 60  0000 C CNN
+F 0 "D7" H 1900 7400 60  0000 C CNN
 F 1 "7SEGMENTS" H 1900 6400 60  0000 C CNN
 F 2 "" H 1900 6850 60  0000 C CNN
@@
 SEGDP
 $Comp
-L 7SEGMENTS AFF8
+L 7SEGMENTS D8
 U 1 1 537131B4
 P 4050 6850
-F 0 "AFF8" H 4050 7400 60  0000 C CNN
+F 0 "D8" H 4050 7400 60  0000 C CNN
 F 1 "7SEGMENTS" H 4050 6400 60  0000 C CNN
 F 2 "" H 4050 6850 60  0000 C CNN
